File: MCU datalogger/mcu datalogger/mcu datalogger.kicad_sch (KiCad schematic)
At the start: 25 parts, among them U1 24LC1025, U2 DS1337S_, U3 24LC1025, U4 ATMEGA328P-AU, Y1 32.768 KHz, Y2 16MHz

Commit message: Completed 2 layer PCB project.
Connections:
- net SCL: no longer R5.2, U4.17 (PB5)
- new net SCK: R5.2, U4.17 (PB5)
Other:
- sheet Connectors ports: added SCK; removed none
Changed lines of the file:
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@@
+    (stroke (width 0) (type default))
+  )
+  (wire (pts (xy 139.7 138.43) (xy 139.7 139.7))
     (stroke (width 0) (type default))
   )
@@
     (stroke (width 0) (type default))
   )
+  (wire (pts (xy 139.7 140.97) (xy 139.7 142.24))
+    (stroke (width 0) (type default))
+  )
   (wire (pts (xy 162.56 44.45) (xy 143.51 44.45))
     (stroke (width 0) (type default))
@@
     (effects (font (size 1.27 1.27)) (justify left bottom))
   )
-  (label "TX" (at 139.7 139.7 180) (fields_autoplaced)
+  (label "TX" (at 139.7 138.43 180) (fields_autoplaced)
     (effects (font (size 1.27 1.27)) (justify right bottom))
   )
@@
     (effects (font (size 1.27 1.27)) (justify right bottom))
   )
-  (label "RX" (at 139.7 142.24 180) (fields_autoplaced)
+  (label "RX" (at 139.7 140.97 180) (fields_autoplaced)
     (effects (font (size 1.27 1.27)) (justify right bottom))
   )
@@
     (effects (font (size 1.27 1.27)) (justify right bottom))
   )
-  (label "SCL" (at 190.5 60.96 180) (fields_autoplaced)
+  (label "SCK" (at 190.5 60.96 180) (fields_autoplaced)
     (effects (font (size 1.27 1.27)) (justify right bottom))
   )
@@
   (label "D7" (at 162.56 140.97 0) (fields_autoplaced)
     (effects (font (size 1.27 1.27)) (justify left bottom))
+  )
+  (label "SCK" (at 139.7 144.78 180) (fields_autoplaced)
+    (effects (font (size 1.27 1.27)) (justify right bottom))
   )
   (label "Vcc" (at 29.21 132.08 180) (fields_autoplaced)
@@
       (effects (font (size 1.27 1.27)) (justify left))
     )
-    (pin "TX" output (at 139.7 139.7 180)
-      (effects (font (size 1.27 1.27)) (justify left))
-    )
-    (pin "RX" input (at 139.7 142.24 180)
+    (pin "TX" output (at 139.7 138.43 180)
+      (effects (font (size 1.27 1.27)) (justify left))
+    )
+    (pin "RX" input (at 139.7 140.97 180)
       (effects (font (size 1.27 1.27)) (justify left))
     )
@@
       (effects (font (size 1.27 1.27)) (justify left))
     )
+    (pin "SCK" passive (at 139.7 144.78 180)
+      (effects (font (size 1.27 1.27)) (justify left))
+    )
