File: MCU datalogger/mcu datalogger/mcu datalogger.kicad_pcb (KiCad board)
At the start: 2 copper layers, 50.3 x 32 mm, 29 parts, among them J1 Conn_01x04_Pin, J2 Conn_01x09_Pin, J3 Conn_01x04_Pin, J4 Conn_02x03_Odd_Even, U1 24LC1025, U2 DS1337S_, U3 24LC1025, U4 ATMEGA328P-AU, Y1 32.768 KHz, Y2 16MHz

Commit message: Modified.
Other:
- board text added: "BOARD CHARACTISTICS :"
- board text added: "Board thickness : 1.6 mm Min hole diameter : 0.3000 mm Impedance control : No Plated board edge : No"
- board text added: "Copper layer count : 2 Board Overall dimension : 32.3 mm x 50.47 mm Min track/spacing : 0.2000 mm / 0.0000 mm Copper finish : None Castellated pads : No"
Changed lines of the file:
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@@
     (pad "2" smd rect (at 2.6 0) (size 3.5 2.4) (layers "F.Cu" "F.Paste" "F.Mask")
       (net 3 "Net-(U4-PB6)") (pinfunction "2") (pintype "passive"))
-    (model "${KICAD6_3DMODEL_DIR}/Crystal.3dshapes/Crystal_SMD_5032-2Pin_5.0x3.2mm_HandSoldering.wrl"
+    (model ":KICAD7_3DMODEL_DIR:Crystal.3dshapes/Crystal_SMD_0603-4Pin_6.0x3.5mm.wrl"
       (offset (xyz 0 0 0))
       (scale (xyz 1 1 1))
@@
     (pad "32" smd roundrect (at -2.8 -4.17) (size 0.55 1.47) (layers "F.Cu" "F.Paste" "F.Mask") (roundrect_rratio 0.18)
       (net 10 "/D2") (pinfunction "PD2") (pintype "bidirectional") (solder_mask_margin 0.102))
+    (model ":KICAD7_3DMODEL_DIR:Package_QFP.3dshapes/TQFP-32_7x7mm_P0.8mm.step"
+      (offset (xyz 0 0 0))
+      (scale (xyz 1 1 1))
+      (rotate (xyz 0 0 0))
+    )
   )
   (footprint "Capacitor_SMD:C_0805_2012Metric" (layer "F.Cu")
@@
     (pad "8" smd roundrect (at 2.475 -1.905) (size 1.97 0.59) (layers "F.Cu" "F.Paste" "F.Mask") (roundrect_rratio 0.07)
       (net 2 "/Vcc") (pinfunction "VCC") (pintype "power_in") (solder_mask_margin 0.102))
+    (model ":KICAD7_3DMODEL_DIR:Package_SO.3dshapes/SO-8_3.9x4.9mm_P1.27mm.wrl"
+      (offset (xyz 0 0 0))
+      (scale (xyz 1 1 1))
+      (rotate (xyz 0 0 0))
+    )
   )
   (footprint "Resistor_SMD:R_0805_2012Metric" (layer "F.Cu")
@@
     (pad "2" smd rect (at 2.6 0 90) (size 3.5 2.4) (layers "F.Cu" "F.Paste" "F.Mask")
       (net 24 "Net-(U2-X1)") (pinfunction "2") (pintype "passive"))
-    (model "${KICAD6_3DMODEL_DIR}/Crystal.3dshapes/Crystal_SMD_5032-2Pin_5.0x3.2mm_HandSoldering.wrl"
+    (model ":KICAD7_3DMODEL_DIR:Crystal.3dshapes/Crystal_SMD_0603-4Pin_6.0x3.5mm.wrl"
       (offset (xyz 0 0 0))
       (scale (xyz 1 1 1))
@@
     (effects (font (size 0.8 0.8) (thickness 0.15)) (justify left bottom))
   )
+  (gr_text "Copper layer count : 2\n\nBoard Overall dimension : 32.3 mm x 50.47 mm\n\nMin track/spacing : 0.2000 mm / 0.0000 mm\n\nCopper finish : None\n\nCastellated pads : No" (at 177.165 87.3252) (layer "Edge.Cuts")
+    (effects (font (size 1 1) (thickness 0.15)) (justify left bottom))
+  )
+  (gr_text "Board thickness : 1.6 mm\n\n\n\nMin hole diameter : 0.3000 mm\n\nImpedance control : No\n\nPlated board edge : No" (at 219.1258 87.1982) (layer "Edge.Cuts")
+    (effects (font (size 1 1) (thickness 0.15)) (justify left bottom))
+  )
+  (gr_text "BOARD CHARACTISTICS :" (at 176.6824 70.485) (layer "Edge.Cuts")
+    (effects (font (size 1.5 2) (thickness 0.375) bold) (justify left bottom))
+  )
+  (dimension (type aligned) (layer "Edge.Cuts")
+    (pts (xy 102.1334 102.616) (xy 152.6032 102.6414))
+    (height 2.911578)
+    (gr_text "50.4698 mm" (at 127.367414 104.390278 359.9711647) (layer "Edge.Cuts")
+      (effects (font (size 1 1) (thickness 0.15)))
+    )
+    (format (prefix "") (suffix "") (units 3) (units_format 1) (precision 4))
+    (style (thickness 0.1) (arrow_length 1.27) (text_position_mode 0) (extension_height 0.58642) (extension_offset 0.5) keep_text_aligned)
+  )
+  (dimension (type aligned) (layer "Edge.Cuts")
+    (pts (xy 96.2914 98.2472) (xy 96.266 65.9384))
+    (height 0.184088)
+    (gr_text "32.3088 mm" (at 97.612788 82.091751 -89.95495616) (layer "Edge.Cuts")
+      (effects (font (size 1 1) (thickness 0.15)))
+    )
+    (format (prefix "") (suffix "") (units 3) (units_format 1) (precision 4))
+    (style (thickness 0.1) (arrow_length 1.27) (text_position_mode 0) (extension_height 0.58642) (extension_offset 0.5) keep_text_aligned)
+  )
   (segment (start 111.2232 80.1072) (end 111.741373 80.1072) (width 0.35) (layer "F.Cu") (net 1))
