File: ANC/ANC_first_PCB.kicad_pcb (KiCad board)
At the start: 2 copper layers, 84 x 41.9 mm, 83 parts, among them J1 Screw_Terminal_01x04, J10 Conn_01x03, J11 Conn_01x03, J12 Conn_01x03, J13 Conn_01x03, J2 Screw_Terminal_01x02, J3 SJ2-35894B-SMT-TR, J4 Conn_01x04, J5 Conn_01x04, J6 Conn_01x06, J7 Conn_01x04, J8 Conn_01x04, J9 Conn_01x04, U1 ICS-40730, U10 LD39015M12R, U2 MAX98090AETL_T, U3 ICS-40730, U4 CMM-3729AB-38308-TR, U5 CMM-3729AB-38308-TR, U6 TLV172IDCK, U7 TLV172IDCK, U8 LD1117S12TR_SOT223, U9 LD39015M18R, Y1 ASE-12.288MHZ-LC-T, x1 0, x2 0

Commit message: Updated ANC.
Other:
- board text removed: "0.0000 mm / 0.0000 mm"
- board text removed: "0.3000 mm"
- board text removed: "1.6000 mm"
- board text removed: "2"
- board text removed: "84.0438 mm x 41.9150 mm"
- board text removed: "BOARD CHARACTERISTICS"
- board text removed: "Board Thickness:"
- board text removed: "Board overall dimensions:"
- board text removed: "Castellated pads:"
- board text removed: "Copper Finish:"
- board text removed: "Copper Layer Count:"
- board text removed: "Edge card connectors:"
- board text removed: "Impedance Control:"
- board text removed: "Min hole diameter:"
- board text removed: "Min track/spacing:"
- board text removed: "No"
- board text removed: "None"
- board text removed: "Plated Board Edge:"
