File: Power supply pcb/Power supply pcb.kicad_pcb (KiCad board)
At the start: 2 copper layers, 30 x 52.8 mm, 18 parts, among them J1 Barrel_Jack_Switch, J2 Conn_01x03_Pin, J3 Conn_01x02_Pin, J4 Screw_Terminal_01x02, J5 Conn_01x03_Pin, J6 Conn_01x02_Pin, J7 Screw_Terminal_01x02, U1 LM317_TO-220, U2 LM7805_TO220

Commit message: Optimized.
Routing:
- net Net-(U1-ADJ): track 41.2 -> 38.2 mm
- net /PWR_OUT_TOP: track 22.8 -> 25.5 mm
- net /12V: track 51.2 -> 49.9 mm
- net /PWR_OUT_BOT: track 23.6 -> 24.6 mm
- added copper zone on F.Cu, net GND
